Commit message: add camera to dron igs.

File: flypulator_description/urdf/hexarotor_igs.urdf (robot description, URDF)
Before this commit: robot drone, 21 links, 20 joints
Links:
- added link camera_link
- added link camera_link_optical
Joints:
- added joint camera_joint: type fixed, parent base_link, child camera_link, origin xyz=0 0 0 rpy=0 0 0, axis 0 1 0
- added joint camera_optical_joint: type fixed, parent camera_link, child camera_link_optical, origin xyz=0 0 0 rpy=-1.5708 0 -1.5708

Commit message: [traj_generator] urdf-> mass adjusted

File: flypulator_description/urdf/hexarotor_igs.urdf (robot description, URDF)
Before this commit: robot drone, 21 links, 20 joints
Links:
- link base_link: mass 3.2461 -> 1.4905
