Commit message: Putting all urdf models in one directory

File: flypulator_description/urdf/hexatilt.xacro (robot description, xacro)
@@ -91,5 +91,5 @@
 <!-- [kg.m^2] [kg.m^2] [kg.m^2] [kg.m^2] [kg.m^2] [kg.m^2] -->
   <!-- Included URDF Files -->
-  <xacro:include filename="$(find flypulator_description_new)/urdf/multirotor_base.xacro" />
+  <xacro:include filename="$(find flypulator_description)/urdf/multirotor_base.xacro" />
   <!-- Instantiate multirotor_base_macro once -->
   <xacro:multirotor_base_macro

File: flypulator_description/urdf/hexatilt_base.xacro (robot description, xacro)
@@ -24,9 +24,9 @@
   <xacro:arg name='log_file' default='hexatilt' />
   <!-- macros for gazebo plugins, sensors -->
-  <!-- <xacro:include filename="$(find flypulator_description_new)/urdf/component_snippets.xacro" /> -->
+  <!-- <xacro:include filename="$(find flypulator_description)/urdf/component_snippets.xacro" /> -->
   <!-- macros for gazebo plugins, for flypulator -->
-  <!-- <xacro:include filename="$(find flypulator_description_new)/urdf/gazebo_plugins.xacro" /> -->
+  <!-- <xacro:include filename="$(find flypulator_description)/urdf/gazebo_plugins.xacro" /> -->
   <!-- Instantiate hexatilt "mechanics" -->
-  <xacro:include filename="$(find flypulator_description_new)/urdf/hexatilt.xacro" />
+  <xacro:include filename="$(find flypulator_description)/urdf/hexatilt.xacro" />
   <xacro:if value="$(arg use_px4_plugins)">
   <xacro:if value="$(arg enable_wind)">

File: flypulator_description/urdf/multirotor_base.xacro (robot description, xacro)
@@ -35,5 +35,5 @@
         <origin xyz="0 0 0" rpy="0 0 0" />
         <geometry>
-          <mesh filename="package://flypulator_description_new/meshes/${mesh_file}"
+          <mesh filename="package://flypulator_description/meshes/${mesh_file}"
             scale="${mesh_scale}" />
           <!-- <box size="${body_width} ${body_width} ${body_height}"/> --> <!-- [m] [m] [m] -->
@@ -95,5 +95,5 @@
         <geometry>
           <!-- <cylinder length="0.005" radius="${radius_rotor}"/> --> <!-- [m] -->
-          <mesh filename="package://flypulator_description_new/meshes/${mesh}_${direction}.dae"
+          <mesh filename="package://flypulator_description/meshes/${mesh}_${direction}.dae"
             scale="${mesh_scale}" />
           <!-- <box size="${2*radius_rotor} 0.01 0.005"/> -->
@@ -164,5 +164,5 @@
         <geometry>
           <!-- <cylinder length="0.005" radius="${radius_rotor}"/> --> <!-- [m] -->
-          <mesh filename="package://flypulator_description_new/meshes/right_leg.dae"
+          <mesh filename="package://flypulator_description/meshes/right_leg.dae"
              scale="${mesh_scale}" />
             <!-- <cylinder length="${length_leg}" radius="${radius_leg}" /> <1 [m] -1> -->
@@ -191,5 +191,5 @@
         <!-- <geometry> -->
           <!-- <cylinder length="0.005" radius="${radius_rotor}"/> --> <!-- [m] -->
-          <!-- <mesh filename="package://flypulator_description_new/meshes/${mesh}_${suffix}.dae" -->
+          <!-- <mesh filename="package://flypulator_description/meshes/${mesh}_${suffix}.dae" -->
             <!-- scale="${mesh_scale}" /> -->
             <!-- <cylinder length="${length_leg}" radius="${radius_leg}" />  -->

Commit message: reading frone parameters from yaml

File: flypulator_description/urdf/hexatilt.xacro (robot description, xacro)
@@ -1,46 +1,48 @@
 <?xml version="1.0"?>
 <robot name="hexatilt" xmlns:xacro="http://ros.org/wiki/xacro">
-  <!-- Properties -->
+  <!--  Convenience Parameters -->
+  <xacro:property name="DP" value="${load_yaml('../param/drone_parameter.yaml')}"/>
   <xacro:property name="namespace" value="/drone" />
   <xacro:property name="PI" value="3.1415926535897931"/>
   <xacro:property name="deg_to_rad" value="0.017453278"/>
   <xacro:property name="to_kgm2" value="1e-9"/>
-  <xacro:property name="rotor_tilt_angle" value="13.6"/> <!--in [deg]-->
-  <xacro:property name="rotor_velocity_slowdown_sim" value="10" />
+  <xacro:property name="sin30" value="0.5" />
+  <xacro:property name="cos30" value="0.866025403784" />
+  <xacro:property name="sqrt2" value="1.4142135623730951" />
+  <!-- Mesh parameters -->
   <xacro:property name="mesh_file" value="hexatilt.dae" />
   <xacro:property name="mesh_scale" value="1 1 1"/>
   <xacro:property name="mesh_scale_prop" value="0.098 0.098 0.098"/>
-  <xacro:property name="mass" value="4.5" /> <!-- [kg] -->
-  <xacro:property name="body_width" value="0.45" /> <!-- [m] -->
-  <xacro:property name="body_height" value="0.085" /> <!-- [m] -->
-  <xacro:property name="mass_rotor" value="0.010" /> <!-- [kg] -->
-  <xacro:property name="arm_length_front_x" value="0.22" /> <!-- [m] -->
-  <xacro:property name="arm_length_back_x" value="0.22" /> <!-- [m] -->
-  <xacro:property name="arm_length_front_y" value="0.37" /> <!-- [m] -->
-  <xacro:property name="arm_length_back_y" value="0.37" /> <!-- [m] -->
-  <!--Added for Hexacopter -->
-  <xacro:property name="arm_length_side_x" value="0.43" /> <!-- [m] -->
-  <xacro:property name="arm_length_side_y" value="0.01" /> <!-- [m] -->
-  <xacro:property name="leg_pos_side_x" value="0.11" /> <!-- [m] -->
-  <xacro:property name="mass_leg" value="0.180" /> <!-- [kg] -->
-  <xacro:property name="radius_leg" value="0.0125" /> <!-- [m] -->
-  <xacro:property name="length_leg" value="0.413" /> <!-- [m] -->
+  <xacro:property name="mesh_scale_leg" value="0.1 0.1 0.1"/>
+  <!-- Geometric Parameters -->
+  <!-- These parameters are pulled from the .yaml file -->
+  <xacro:property name="rotor_tilt_angle"   value="${DP['uav/alpha']}"/> <!--in [deg]-->
+  <xacro:property name="body_radius"        value="${DP['uav/body_radius']}" /> <!-- [m] -->
+  <xacro:property name="body_height"        value="${DP['uav/body_height']}" />
+  <xacro:property name="mass_rotor"         value="${DP['uav/mass_rotor']}" /> <!-- [kg] -->
+  <xacro:property name="arm_length_x"       value="${DP['uav/x']}" /> <!-- [Man[m] -->
+  <xacro:property name="arm_length_y"       value="${DP['uav/y']}" /> <!-- [m] -->
+  <xacro:property name="arm_length_side_x"  value="${DP['uav/side_x']}" /> <!-- [m] -->
+  <xacro:property name="arm_length_side_y"  value="${DP['uav/side_y']}" /> <!-- [m] -->
+  <xacro:property name="radius_leg"         value="${DP['uav/leg_radius']}" /> <!--[Man [m] -->
+  <xacro:property name="length_leg"         value="${DP['uav/leg_length']}" /> <!-- [m] -->
+  <xacro:property name="rotor_offset_top"   value="${DP['uav/blade_offset_top']}"/> <!-- [m] -->
+  <xacro:property name="radius_rotor"       value="${DP['uav/blade_radius']}" /> <!-- [[Manm] -->
+   <!-- Simulation Properties -->[Ma
   <xacro:property name="max_leg_velocity" value="0.10" /> <!-- [m] -->
-  <xacro:property name="mesh_scale_leg" value="0.1 0.1 0.1"/>
-  <!--#################### -->
-  <xacro:property name="rotor_offset_top" value="0.06" /> <!-- [m] -->
-  <xacro:property name="radius_rotor" value="0.1905" /> <!-- [m] -->
-  <xacro:property name="motor_constant" value="8.54858e-06" /> <!-- [kg.m/s^2] -->
+  <xacro:property name="rotor_velocity_slowdown_sim" value="10" />
+    <xacro:property name="motor_constant" value="8.54858e-06" /> <!-- [kg.m/s^2] -->
   <xacro:property name="moment_constant" value="0.06" /> <!-- [m] -->
   <xacro:property name="time_constant_up" value="0.0125" /> <!-- [s] -->
   <xacro:property name="time_constant_down" value="0.025" /> <!-- [s] -->
   <xacro:property name="max_rot_velocity" value="1100" /> <!-- [rad/s] -->
-  <xacro:property name="sin30" value="0.5" />
-  <xacro:property name="cos30" value="0.866025403784" />
-  <xacro:property name="sqrt2" value="1.4142135623730951" />
   <xacro:property name="rotor_drag_coefficient" value="8.06428e-04" />
   <xacro:property name="rolling_moment_coefficient" value="0.000001" />
   <xacro:property name="color" value="DarkGrey" />
   <!-- Property Blocks -->
+ <!-- Mass and inertial Properties -->
+  <xacro:property name="base_mass" value="${DP['uav/mass']}" /> <!-- [kg] -->
+  <xacro:property name="leg_pos_side_x" value="0.11" /> <!-- [m] -->
+  <xacro:property name="mass_leg" value="0.180" /> <!-- [kg] -->
 <!-- Moment of Inertia at Origin   (g mm^2) -->
   <xacro:property name="body_inertia">
@@ -56,5 +58,16 @@
 	izz = "${ 2.429E+08 *to_kgm2}"     />
     </xacro:property>
-<!-- Moment of Inertia at Center of Mass   (g mm^2) -->
+  <xacro:property name="leg_inertia">
+    <inertia
+      ixx = "${ 3.321E+06*to_kgm2 }"
+      ixy = "${ 0.048    *to_kgm2 }"
+      ixz = "${ 4.097E+05*to_kgm2 }"
+      iyx = "${ 0.048    *to_kgm2 }"
+      iyy = "${ 2.407E+06*to_kgm2 }"
+      iyz = "${ -0.271    *to_kgm2 }"
+      izx = "${ 4.097E+05*to_kgm2 }"
+      izy = "${ -0.271   *to_kgm2 }"
+      izz = "${ 1.070E+06*to_kgm2 }"/>
+     </xacro:property>
   <xacro:property name="rotor_inertia">
     <inertia
@@ -69,37 +82,15 @@
     iyz = "${ -1.849E+0*to_kgm2 }"/>
 	  </xacro:property>
-  <!-- <xacro:property name="body_inertia"> -->
-      <!-- <inertia
-           ixx="0.0347563"
-           ixy="0.0"
-           ixz="0.0"
-           iyy="0.0458929"
-           iyz="0.0"
-           izz="0.0977" /> -->
-  <!-- [kg.m^2] [kg.m^2] [kg.m^2] [kg.m^2] [kg.m^2] [kg.m^2] -->
-  <!-- </xacro:property> -->
-  <!-- inertia of a single rotor, assuming it is a cuboid. Height=3mm, width=15mm -->
-  <!-- <xacro:property name="rotor_inertia"> -->
-  <!--   <inertia -->
-  <!--   ixx="${1/12 * mass_rotor * (0.015 * 0.015 + 0.003 * 0.003) * rotor_velocity_slowdown_sim}" -->
-  <!--   iyy="${1/12 * mass_rotor * (4 * radius_rotor * radius_rotor + 0.003 * 0.003) * rotor_velocity_slowdown_sim}" -->
-  <!--   izz="${1/12 * mass_rotor * (4 * radius_rotor * radius_rotor + 0.015 * 0.015) * rotor_velocity_slowdown_sim}" -->
-  <!--   ixy="0.0" -->
-  <!--   ixz="0.0" -->
-  <!--   iyz="0.0" /> -->
-  <!-- </xacro:property> -->
-<!-- [kg.m^2] [kg.m^2] [kg.m^2] [kg.m^2] [kg.m^2] [kg.m^2] -->
-  <!-- Included URDF Files -->
+    <!-- Included URDF Files -->
   <xacro:include filename="$(find flypulator_description)/urdf/multirotor_base.xacro" />
   <!-- Instantiate multirotor_base_macro once -->
   <xacro:multirotor_base_macro
     robot_namespace="${namespace}"
-    mass="${mass}"
-    body_width="${body_width}"
+    mass="${base_mass}"
+    body_radius="${body_radius}"
     body_height="${body_height}"
     mesh_file="${mesh_file}"
     mesh_scale="${mesh_scale}"
-    color="${color}"
-    >
+    color="${color}">
     <xacro:insert_block name="body_inertia" />
   </xacro:multirotor_base_macro>
@@ -123,5 +114,5 @@
     mesh_scale="${mesh_scale_prop}"
     color="DarkGrey">
-    <origin xyz="${arm_length_front_x+0.01} -${arm_length_front_y} ${rotor_offset_top}" rpy="${rotor_tilt_angle*deg_to_rad} 0  ${120*deg_to_rad}" />
+    <origin xyz="${arm_length_x+0.01} -${arm_length_y} ${rotor_offset_top}" rpy="${rotor_tilt_angle*deg_to_rad} 0  ${120*deg_to_rad}" />
     <xacro:insert_block name="rotor_inertia" />
   </xacro:vertical_rotor>
@@ -144,5 +135,5 @@
     mesh_scale="${mesh_scale_prop}"
     color="Red">
-    <origin xyz="-${arm_length_back_x-0.02} ${arm_length_back_y} ${rotor_offset_top}" rpy="-${rotor_tilt_angle*deg_to_rad} 0  -${60*deg_to_rad}" />
+    <origin xyz="-${arm_length_x-0.02} ${arm_length_y} ${rotor_offset_top}" rpy="-${rotor_tilt_angle*deg_to_rad} 0  -${60*deg_to_rad}" />
     <xacro:insert_block name="rotor_inertia" />
   </xacro:vertical_rotor>
@@ -164,5 +155,5 @@
     mesh_scale="${mesh_scale_prop}"
     color="Red">
-    <origin xyz="${arm_length_front_x-0.02} ${arm_length_front_y} ${rotor_offset_top}" rpy= "${rotor_tilt_angle*deg_to_rad} 0  ${240*deg_to_rad}"/>
+    <origin xyz="${arm_length_x-0.02} ${arm_length_y} ${rotor_offset_top}" rpy= "${rotor_tilt_angle*deg_to_rad} 0  ${240*deg_to_rad}"/>
     <xacro:insert_block name="rotor_inertia" />
   </xacro:vertical_rotor>
@@ -184,5 +175,5 @@
     mesh_scale="${mesh_scale_prop}"
     color="DarkGrey">
-    <origin xyz="-${arm_length_back_x+0.01} -${arm_length_back_y} ${rotor_offset_top}" rpy= "-${rotor_tilt_angle*deg_to_rad} 0  ${60*deg_to_rad}"/>
+    <origin xyz="-${arm_length_x+0.01} -${arm_length_y} ${rotor_offset_top}" rpy= "-${rotor_tilt_angle*deg_to_rad} 0  ${60*deg_to_rad}"/>
     <xacro:insert_block name="rotor_inertia" />
   </xacro:vertical_rotor>
@@ -240,5 +231,5 @@
     reflect="-1">
     <origin xyz="${leg_pos_side_x} 0 -0.02" rpy="0 -${10*deg_to_rad} 0" />
-    <xacro:insert_block name="rotor_inertia" />
+    <xacro:insert_block name="leg_inertia" />
   </xacro:landing_gear>
 <xacro:landing_gear robot_namespace="${namespace}"
@@ -255,5 +246,5 @@
     color="DarkGrey">
     <origin xyz="-${leg_pos_side_x} 0 -0.02" rpy="0 ${10*deg_to_rad} 0" />
-    <xacro:insert_block name="rotor_inertia" />
+    <xacro:insert_block name="leg_inertia" />
   </xacro:landing_gear>
   <!--<gazebo>

File: flypulator_description/urdf/multirotor_base.xacro (robot description, xacro)
@@ -19,5 +19,5 @@
   <!-- Main multirotor link -->
   <xacro:macro name="multirotor_base_macro"
-    params="robot_namespace mass body_width body_height mesh_file mesh_scale color *inertia">
+    params="robot_namespace mass body_radius body_height mesh_file mesh_scale color *inertia">
     <link name="base_link"></link>
     <joint name="base_joint" type="fixed">
@@ -37,5 +37,4 @@
           <mesh filename="package://flypulator_description/meshes/${mesh_file}"
             scale="${mesh_scale}" />
-          <!-- <box size="${body_width} ${body_width} ${body_height}"/> --> <!-- [m] [m] [m] -->
         </geometry>
       </visual>
@@ -43,6 +42,5 @@
         <origin xyz="0 0 0" rpy="0 0 0" />
         <geometry>
-            <cylinder length="${body_height}" radius="${body_width}" /> <!-- [m] -->
-          <!--box size="${body_width} ${body_width} ${body_height}" /--> <!-- [m] [m] [m] -->
+            <cylinder length="${body_height}" radius="${body_radius}" /> <!-- [m] -->
         </geometry>
       </collision>
@@ -107,20 +105,20 @@
     </link>
     <gazebo>
-      <plugin name="${suffix}_motor_model" filename="librotors_gazebo_motor_model.so">
-        <robotNamespace>${robot_namespace}</robotNamespace>
-        <jointName>rotor_${motor_number}_joint</jointName>
-        <linkName>rotor_${motor_number}</linkName>
-        <turningDirection>${direction}</turningDirection>
-        <timeConstantUp>${time_constant_up}</timeConstantUp>
-        <timeConstantDown>${time_constant_down}</timeConstantDown>
-        <maxRotVelocity>${max_rot_velocity}</maxRotVelocity>
-        <motorConstant>${motor_constant}</motorConstant>
-        <momentConstant>${moment_constant}</momentConstant>
-        <commandSubTopic>/gazebo/command/motor_speed</commandSubTopic>
-        <motorNumber>${motor_number}</motorNumber>
-        <rotorDragCoefficient>${rotor_drag_coefficient}</rotorDragCoefficient>
-        <rollingMomentCoefficient>${rolling_moment_coefficient}</rollingMomentCoefficient>
-        <motorSpeedPubTopic>/motor_speed/${motor_number}</motorSpeedPubTopic>
-        <rotorVelocitySlowdownSim>${rotor_velocity_slowdown_sim}</rotorVelocitySlowdownSim>
+      <!-- <plugin name="${suffix}_motor_model" filename="librotors_gazebo_motor_model.so"> -->
+      <!--   <robotNamespace>${robot_namespace}</robotNamespace> -->
+      <!--   <jointName>rotor_${motor_number}_joint</jointName> -->
+      <!--   <linkName>rotor_${motor_number}</linkName> -->
+      <!--   <turningDirection>${direction}</turningDirection> -->
+      <!--   <timeConstantUp>${time_constant_up}</timeConstantUp> -->
+      <!--   <timeConstantDown>${time_constant_down}</timeConstantDown> -->
+      <!--   <maxRotVelocity>${max_rot_velocity}</maxRotVelocity> -->
+      <!--   <motorConstant>${motor_constant}</motorConstant> -->
+      <!--   <momentConstant>${moment_constant}</momentConstant> -->
+      <!--   <commandSubTopic>/gazebo/command/motor_speed</commandSubTopic> -->
+      <!--   <motorNumber>${motor_number}</motorNumber> -->
+      <!--   <rotorDragCoefficient>${rotor_drag_coefficient}</rotorDragCoefficient> -->
+      <!--   <rollingMomentCoefficient>${rolling_moment_coefficient}</rollingMomentCoefficient> -->
+      <!--   <motorSpeedPubTopic>/motor_speed/${motor_number}</motorSpeedPubTopic> -->
+      <!--   <rotorVelocitySlowdownSim>${rotor_velocity_slowdown_sim}</rotorVelocitySlowdownSim> -->
         <!--
         <gazebo_joint_control_pid>
@@ -134,5 +132,5 @@
         </gazebo_joint_control_pid>
       -->
-      </plugin>
+      <!-- </plugin> -->
     </gazebo>
     <gazebo reference="rotor_${motor_number}">

Commit message: checkout to switch branch

File: flypulator_description/urdf/hexatilt.xacro (robot description, xacro)
@@ -20,5 +20,5 @@
   <xacro:property name="body_radius"        value="${DP['uav/body_radius']}" /> <!-- [m] -->
   <xacro:property name="body_height"        value="${DP['uav/body_height']}" />
-  <xacro:property name="mass_rotor"         value="${DP['uav/mass_rotor']}" /> <!-- [kg] -->
+  <xacro:property name="mass_rotor"         value="${DP['uav/blade_mass']}" /> <!-- [kg] -->
   <xacro:property name="arm_length_x"       value="${DP['uav/x']}" /> <!-- [Man[m] -->
   <xacro:property name="arm_length_y"       value="${DP['uav/y']}" /> <!-- [m] -->
@@ -29,8 +29,8 @@
   <xacro:property name="rotor_offset_top"   value="${DP['uav/blade_offset_top']}"/> <!-- [m] -->
   <xacro:property name="radius_rotor"       value="${DP['uav/blade_radius']}" /> <!-- [[Manm] -->
-   <!-- Simulation Properties -->[Ma
+   <!-- Simulation Properties -->
   <xacro:property name="max_leg_velocity" value="0.10" /> <!-- [m] -->
   <xacro:property name="rotor_velocity_slowdown_sim" value="10" />
-    <xacro:property name="motor_constant" value="8.54858e-06" /> <!-- [kg.m/s^2] -->
+  <xacro:property name="motor_constant" value="8.54858e-06" /> <!-- [kg.m/s^2] -->
   <xacro:property name="moment_constant" value="0.06" /> <!-- [m] -->
   <xacro:property name="time_constant_up" value="0.0125" /> <!-- [s] -->
@@ -60,13 +60,13 @@
   <xacro:property name="leg_inertia">
     <inertia
-      ixx = "${ 3.321E+06*to_kgm2 }"
-      ixy = "${ 0.048    *to_kgm2 }"
-      ixz = "${ 4.097E+05*to_kgm2 }"
-      iyx = "${ 0.048    *to_kgm2 }"
-      iyy = "${ 2.407E+06*to_kgm2 }"
-      iyz = "${ -0.271    *to_kgm2 }"
-      izx = "${ 4.097E+05*to_kgm2 }"
-      izy = "${ -0.271   *to_kgm2 }"
-      izz = "${ 1.070E+06*to_kgm2 }"/>
+    ixx = "${ 3.321E+06*to_kgm2 }"
+    ixy = "${ 0.048    *to_kgm2 }"
+    ixz = "${ 4.097E+05*to_kgm2 }"
+    iyx = "${ 0.048    *to_kgm2 }"
+    iyy = "${ 2.407E+06*to_kgm2 }"
+    iyz = "${ -0.271    *to_kgm2 }"
+    izx = "${ 4.097E+05*to_kgm2 }"
+    izy = "${ -0.271   *to_kgm2 }"
+    izz = "${ 1.070E+06*to_kgm2 }"/>
      </xacro:property>
   <xacro:property name="rotor_inertia">
