Commit message: updated motor numbers and position

File: flypulator_description/urdf/hexatilt.xacro (robot description, xacro)
@@ -12,5 +12,5 @@
   <!-- Mesh parameters -->
   <xacro:property name="mesh_file" value="hexatilt.dae" />
-  <xacro:property name="mesh_scale" value="1 1 1"/>
+  <xacro:property name="mesh_scale" value="0.001 0.001 0.001"/>
   <xacro:property name="mesh_scale_prop" value="0.098 0.098 0.098"/>
   <xacro:property name="mesh_scale_leg" value="0.1 0.1 0.1"/>
@@ -18,6 +18,6 @@
   <!-- These parameters are pulled from the .yaml file -->
   <xacro:property name="rotor_tilt_angle"   value="${DP['uav/alpha']}"/> <!--in [deg]-->
-  <xacro:property name="body_radius"        value="${DP['uav/body_radius']}" /> <!-- [m] -->
-  <xacro:property name="body_height"        value="${DP['uav/body_height']}" />
+  <xacro:property name="body_radius"        value="${DP['uav/base_radius']}" /> <!-- [m] -->
+  <xacro:property name="body_height"        value="${DP['uav/base_height']}" />
   <xacro:property name="mass_rotor"         value="${DP['uav/blade_mass']}" /> <!-- [kg] -->
   <xacro:property name="arm_length_x"       value="${DP['uav/x']}" /> <!-- [Man[m] -->
@@ -42,5 +42,5 @@
   <!-- Property Blocks -->
  <!-- Mass and inertial Properties -->
-  <xacro:property name="base_mass" value="${DP['uav/mass']}" /> <!-- [kg] -->
+  <xacro:property name="base_mass" value="${DP['uav/base_mass']}" /> <!-- [kg] -->
   <xacro:property name="leg_pos_side_x" value="0.11" /> <!-- [m] -->
   <xacro:property name="mass_leg" value="0.180" /> <!-- [kg] -->
@@ -96,5 +96,25 @@
   </xacro:multirotor_base_macro>
   <!-- Instantiate rotors -->
-  <xacro:vertical_rotor
+  <xacro:vertical_rotor robot_namespace="${namespace}"
+    suffix="back_right"
+    direction="cw"
+    motor_constant="${motor_constant}"
+    moment_constant="${moment_constant}"
+    parent="base_link"
+    mass_rotor="${mass_rotor}"
+    radius_rotor="${radius_rotor}"
+    time_constant_up="${time_constant_up}"
+    time_constant_down="${time_constant_down}"
+    max_rot_velocity="${max_rot_velocity}"
+    motor_number="1"
+    rotor_drag_coefficient="${rotor_drag_coefficient}"
+    rolling_moment_coefficient="${rolling_moment_coefficient}"
+    mesh="hexatilt_prop"
+    mesh_scale="${mesh_scale_prop}"
+    color="DarkGrey">
+    <origin xyz="-${arm_length_x+0.01} -${arm_length_y} ${rotor_offset_top}" rpy= "-${rotor_tilt_angle*deg_to_rad} 0  ${60*deg_to_rad}"/>
+    <xacro:insert_block name="rotor_inertia" />
+  </xacro:vertical_rotor>
+ <xacro:vertical_rotor
     robot_namespace="${namespace}"
     suffix="front_right"
@@ -108,5 +128,5 @@
     time_constant_down="${time_constant_down}"
     max_rot_velocity="${max_rot_velocity}"
-    motor_number="0"
+    motor_number="2"
     rotor_drag_coefficient="${rotor_drag_coefficient}"
     rolling_moment_coefficient="${rolling_moment_coefficient}"
@@ -115,4 +135,44 @@
     color="DarkGrey">
     <origin xyz="${arm_length_x+0.01} -${arm_length_y} ${rotor_offset_top}" rpy="${rotor_tilt_angle*deg_to_rad} 0  ${120*deg_to_rad}" />
+    <xacro:insert_block name="rotor_inertia" />
+  </xacro:vertical_rotor>
+  <xacro:vertical_rotor robot_namespace="${namespace}"
+    suffix="back_right"
+    direction="cw"
+    motor_constant="${motor_constant}"
+    moment_constant="${moment_constant}"
+    parent="base_link"
+    mass_rotor="${mass_rotor}"
+    radius_rotor="${radius_rotor}"
+    time_constant_up="${time_constant_up}"
+    time_constant_down="${time_constant_down}"
+    max_rot_velocity="${max_rot_velocity}"
+    motor_number="3"
+    rotor_drag_coefficient="${rotor_drag_coefficient}"
+    rolling_moment_coefficient="${rolling_moment_coefficient}"
+    mesh="hexatilt_prop"
+    mesh_scale="${mesh_scale_prop}"
+    color="DarkGrey">
+    <origin xyz="${arm_length_side_x} -${arm_length_side_y} ${rotor_offset_top}" rpy="-${rotor_tilt_angle*deg_to_rad} 0  ${180*deg_to_rad}" />
+    <xacro:insert_block name="rotor_inertia" />
+  </xacro:vertical_rotor>
+  <xacro:vertical_rotor robot_namespace="${namespace}"
+    suffix="front_left"
+    direction="cw"
+    motor_constant="${motor_constant}"
+    moment_constant="${moment_constant}"
+    parent="base_link"
+    mass_rotor="${mass_rotor}"
+    radius_rotor="${radius_rotor}"
+    time_constant_up="${time_constant_up}"
+    time_constant_down="${time_constant_down}"
+    max_rot_velocity="${max_rot_velocity}"
+    motor_number="4"
+    rotor_drag_coefficient="${rotor_drag_coefficient}"
+    rolling_moment_coefficient="${rolling_moment_coefficient}"
+    mesh="hexatilt_prop"
+    mesh_scale="${mesh_scale_prop}"
+    color="Red">
+    <origin xyz="${arm_length_x-0.02} ${arm_length_y} ${rotor_offset_top}" rpy= "${rotor_tilt_angle*deg_to_rad} 0  ${240*deg_to_rad}"/>
     <xacro:insert_block name="rotor_inertia" />
   </xacro:vertical_rotor>
@@ -129,5 +189,5 @@
     time_constant_down="${time_constant_down}"
     max_rot_velocity="${max_rot_velocity}"
-    motor_number="1"
+    motor_number="5"
     rotor_drag_coefficient="${rotor_drag_coefficient}"
     rolling_moment_coefficient="${rolling_moment_coefficient}"
@@ -139,24 +199,4 @@
   </xacro:vertical_rotor>
   <xacro:vertical_rotor robot_namespace="${namespace}"
-    suffix="front_left"
-    direction="cw"
-    motor_constant="${motor_constant}"
-    moment_constant="${moment_constant}"
-    parent="base_link"
-    mass_rotor="${mass_rotor}"
-    radius_rotor="${radius_rotor}"
-    time_constant_up="${time_constant_up}"
-    time_constant_down="${time_constant_down}"
-    max_rot_velocity="${max_rot_velocity}"
-    motor_number="2"
-    rotor_drag_coefficient="${rotor_drag_coefficient}"
-    rolling_moment_coefficient="${rolling_moment_coefficient}"
-    mesh="hexatilt_prop"
-    mesh_scale="${mesh_scale_prop}"
-    color="Red">
-    <origin xyz="${arm_length_x-0.02} ${arm_length_y} ${rotor_offset_top}" rpy= "${rotor_tilt_angle*deg_to_rad} 0  ${240*deg_to_rad}"/>
-    <xacro:insert_block name="rotor_inertia" />
-  </xacro:vertical_rotor>
-  <xacro:vertical_rotor robot_namespace="${namespace}"
     suffix="back_right"
     direction="cw"
@@ -169,25 +209,5 @@
     time_constant_down="${time_constant_down}"
     max_rot_velocity="${max_rot_velocity}"
-    motor_number="3"
-    rotor_drag_coefficient="${rotor_drag_coefficient}"
-    rolling_moment_coefficient="${rolling_moment_coefficient}"
-    mesh="hexatilt_prop"
-    mesh_scale="${mesh_scale_prop}"
-    color="DarkGrey">
-    <origin xyz="-${arm_length_x+0.01} -${arm_length_y} ${rotor_offset_top}" rpy= "-${rotor_tilt_angle*deg_to_rad} 0  ${60*deg_to_rad}"/>
-    <xacro:insert_block name="rotor_inertia" />
-  </xacro:vertical_rotor>
-  <xacro:vertical_rotor robot_namespace="${namespace}"
-    suffix="back_right"
-    direction="cw"
-    motor_constant="${motor_constant}"
-    moment_constant="${moment_constant}"
-    parent="base_link"
-    mass_rotor="${mass_rotor}"
-    radius_rotor="${radius_rotor}"
-    time_constant_up="${time_constant_up}"
-    time_constant_down="${time_constant_down}"
-    max_rot_velocity="${max_rot_velocity}"
-    motor_number="4"
+    motor_number="6"
     rotor_drag_coefficient="${rotor_drag_coefficient}"
     rolling_moment_coefficient="${rolling_moment_coefficient}"
@@ -196,24 +216,4 @@
     color="DarkGrey">
     <origin xyz="-${arm_length_side_x} -${arm_length_side_y} ${rotor_offset_top}" rpy="${rotor_tilt_angle*deg_to_rad} 0  ${0*deg_to_rad}" />
-    <xacro:insert_block name="rotor_inertia" />
-  </xacro:vertical_rotor>
-  <xacro:vertical_rotor robot_namespace="${namespace}"
-    suffix="back_right"
-    direction="cw"
-    motor_constant="${motor_constant}"
-    moment_constant="${moment_constant}"
-    parent="base_link"
-    mass_rotor="${mass_rotor}"
-    radius_rotor="${radius_rotor}"
-    time_constant_up="${time_constant_up}"
-    time_constant_down="${time_constant_down}"
-    max_rot_velocity="${max_rot_velocity}"
-    motor_number="5"
-    rotor_drag_coefficient="${rotor_drag_coefficient}"
-    rolling_moment_coefficient="${rolling_moment_coefficient}"
-    mesh="hexatilt_prop"
-    mesh_scale="${mesh_scale_prop}"
-    color="DarkGrey">
-    <origin xyz="${arm_length_side_x} -${arm_length_side_y} ${rotor_offset_top}" rpy="-${rotor_tilt_angle*deg_to_rad} 0  ${180*deg_to_rad}" />
     <xacro:insert_block name="rotor_inertia" />
   </xacro:vertical_rotor>
@@ -248,8 +248,5 @@
     <xacro:insert_block name="leg_inertia" />
   </xacro:landing_gear>
-  <!--<gazebo>
-    <plugin name="control_plugin" filename="libcontrol_plugin.so">
-    </plugin>
-  </gazebo>-->
+<!-- Gazebo plugins .. move to import document.. -->
   <gazebo>
     <plugin name="fake_sensor_plugin" filename="libfake_sensor_plugin.so">
@@ -262,96 +259,10 @@
   </gazebo>
   <gazebo>
-    <plugin name="drone_internal_imu_plugin" filename="libhector_gazebo_ros_imu.so" >
-      <robotNamespace>${namespace}</robotNamespace>
-      <alwaysOn>true</alwaysOn>
-      <bodyName>base_link</bodyName>
-      <frameName>base_link</frameName>
-      <topicName>IMU/imu_data</topicName>
-      <serviceName>drone/internal_sensors/imu_service</serviceName>
-      <updateRate>100.0</updateRate>
-      <gaussianNoise>0.001</gaussianNoise>
-      <!-- accelerometer params -->
-      <accelOffset>0.0 0.0 0.0</accelOffset>
-      <accelGaussianNoise>0.0003 0.0003 0.0003</accelGaussianNoise>
-      <accelDrift>0.00004 0.00004 0.00004</accelDrift>
-      <accelFrequency>0.0025 0.0025 0.0025</accelFrequency>
-      <!-- gyroscope params -->
-      <rateOffset>0.0 0.0 0.0</rateOffset>
-      <rateDrift>0.01 0.01 0.01</rateDrift>
-      <rateDriftFrequency>0.001 0.001 0.001</rateDriftFrequency>
-      <rateGaussianNoise>0.01 0.01 0.01</rateGaussianNoise>
+    <plugin name="propulsion_plugin" filename="libpropulsion_plugin.so">
     </plugin>
   </gazebo>
-  <gazebo>
-    <plugin name="drone_internal_magnetic_sim" filename="libhector_gazebo_ros_magnetic.so">
-      <robotNamespace>${namespace}</robotNamespace>
-      <updateRate>100.0</updateRate>
-      <bodyName>base_link</bodyName>
-      <frameId>base_link</frameId>
-      <topicName>MAGNET/magnetic_data</topicName>
-      <offset>0 0 0</offset>
-      <drift>0.0 0.0 0.0</drift>
-      <gaussianNoise>1.3e-3 1.3e-3 1.3e-3</gaussianNoise>
-    </plugin>
-  </gazebo>
-  <gazebo>
-    <plugin name="drone_internal_gps_sim" filename="libhector_gazebo_ros_gps.so">
-      <robotNamespace>${namespace}</robotNamespace>
-      <updateRate>4.0</updateRate>
-      <bodyName>base_link</bodyName>
-      <frameId>base_link</frameId>
-      <topicName>GPS/fix</topicName>
-      <velocityTopicName>GPS/fix_velocity</velocityTopicName>
-      <referenceLatitude>49.860246</referenceLatitude>
-      <referenceLongitude>8.687077</referenceLongitude>
-      <drift>0.0 0.0 0.0</drift>
-      <gaussianNoise>0.01 0.01 0.01</gaussianNoise>
-      <velocityDrift>0 0 0</velocityDrift>
-      <velocityGaussianNoise>0.01 0.01 0.01</velocityGaussianNoise>
-    </plugin>
-  </gazebo>
-  <!-- <gazebo reference="base_link"> -->
-  <!--   <sensor type="camera" name="camera1"> -->
-  <!--     <update_rate>30.0</update_rate> -->
-  <!--     <camera name="head"> -->
-  <!--       <vertical_fov>3.1415926</vertical_fov> -->
-  <!--       <image> -->
-  <!--         <width>800</width> -->
-  <!--         <height>800</height> -->
-  <!--         <format>R8G8B8</format> -->
-  <!--       </image> -->
-  <!--       <clip> -->
-  <!--         <near>0.02</near> -->
-  <!--         <far>300</far> -->
-  <!--       </clip> -->
-  <!--       <noise> -->
-  <!--         <type>gaussian</type>  --> -->
-          <!-- Noise is sampled independently per pixel on each frame.
-               That pixel's noise value is added to each of its color
-               channels, which at that point lie in the range [0,1]. -->
-          <!-- <mean>0.0</mean> -->
-          <!-- <stddev>0.007</stddev> -->
-        <!-- </noise> -->
-      <!-- </camera> -->
-      <!-- <plugin name="camera_controller" filename="libgazebo_ros_camera.so"> -->
-        <!-- <robotNamespace>${namespace}</robotNamespace> -->
-        <!-- <alwaysOn>true</alwaysOn> -->
-        <!-- <updateRate>0.0</updateRate> -->
-        <!-- <cameraName>camera1</cameraName> -->
-        <!-- <imageTopicName>image_raw</imageTopicName> -->
-        <!-- <cameraInfoTopicName>camera_info</cameraInfoTopicName> -->
-        <!-- <frameName>base_link</frameName> -->
-        <!-- <hackBaseline>0.07</hackBaseline> -->
-        <!-- <distortionK1>0.0</distortionK1> -->
-        <!-- <distortionK2>0.0</distortionK2> -->
-        <!-- <distortionK3>0.0</distortionK3> -->
-        <!-- <distortionT1>0.0</distortionT1> -->
-        <!-- <distortionT2>0.0</distortionT2> -->
-      <!-- </plugin> -->
-    <!-- </sensor> -->
-  <!-- </gazebo> -->
-<gazebo>
-    <plugin name="propulsion_plugin_hexa" filename="libpropulsion_plugin_hexa.so">
-    </plugin>
-  </gazebo>
+<!-- <gazebo> -->
+<!--     <plugin name="propulsion_plugin_hexa" filename="libpropulsion_plugin_hexa.so"> -->
+<!--     </plugin> -->
+<!--   </gazebo> -->
 </robot>

File: flypulator_description/urdf/multirotor_base.xacro (robot description, xacro)
@@ -1,19 +1,10 @@
 <?xml version="1.0"?>
-<!--
-  Copyright 2015 Fadri Furrer, ASL, ETH Zurich, Switzerland
-  Copyright 2015 Michael Burri, ASL, ETH Zurich, Switzerland
-  Copyright 2015 Mina Kamel, ASL, ETH Zurich, Switzerland
-  Copyright 2015 Janosch Nikolic, ASL, ETH Zurich, Switzerland
-  Copyright 2015 Markus Achtelik, ASL, ETH Zurich, Switzerland
-  Licensed under the Apache License, Version 2.0 (the "License");
-  you may not use this file except in compliance with the License.
-  You may obtain a copy of the License at
-  http://www.apache.org/licenses/LICENSE-2.0
-  Unless required by applicable law or agreed to in writing, software
-  distributed under the License is distributed on an "AS IS" BASIS,
-  WITHOUT WARRANTIES OR CONDITIONS OF ANY KIND, either express or implied.
-  See the License for the specific language governing permissions and
-  limitations under the License.
--->
+<!--  multirotor_base.xacro -->
+ <!-- This file contains the macros for the UAV.
+    The following macros are defined here:
+    * mulitirotor_base_macro
+    * vertical_rotor
+    * landing_gear -->
+    <!-- The gazebo plugins that were used in px4 are located at /src/Firmware/Tools/sitl_gazebo/src. (have to clone their firmware folder) Can be viewed for comparison with our own plugins -->
 <robot xmlns:xacro="http://ros.org/wiki/xacro">
   <!-- Main multirotor link -->
@@ -46,44 +37,21 @@
       </collision>
     </link>
-    <!-- attach multirotor_base_plugin to the base_link -->
+    <!--PX4 memory: attach multirotor_base_plugin to the base_link -->
     <gazebo>
-      <plugin filename="librotors_gazebo_multirotor_base_plugin.so" name="rosbag">
-        <robotNamespace>${robot_namespace}</robotNamespace>
-        <linkName>base_link</linkName>
-        <rotorVelocitySlowdownSim>${rotor_velocity_slowdown_sim}</rotorVelocitySlowdownSim>
-      </plugin>
     </gazebo>
     <gazebo reference="base_link">
-      <material>Gazebo/${color}</material>
-      <collision name='base_link_inertia_collision'>
-        <surface>
-          <contact>
-            <ode>
-              <min_depth>0.001</min_depth>
-              <max_vel>0.0</max_vel>
-            </ode>
-          </contact>
-          <friction>
-            <ode/>
-          </friction>
-        </surface>
-      </collision>
-   </gazebo>
+    <material>Gazebo/${color}</material>
+    </gazebo>
   </xacro:macro>
   <!-- Rotor joint and link -->
   <xacro:macro name="vertical_rotor"
     params="robot_namespace suffix direction motor_constant moment_constant parent mass_rotor radius_rotor time_constant_up time_constant_down max_rot_velocity motor_number rotor_drag_coefficient rolling_moment_coefficient color mesh mesh_scale *origin *inertia">
-    <joint name="rotor_${motor_number}_joint" type="continuous">
+    <joint name="blade_joint_${motor_number}" type="continuous">
       <xacro:insert_block name="origin" />
       <axis xyz="0 0 1" />
-      <!-- TODO(ff): not currently set because it's not yet supported -->
-      <!-- <limit effort="2000" velocity="${max_rot_velocity}" /> -->
       <parent link="${parent}" />
-      <child link="rotor_${motor_number}" />
+      <child link="blade_link_${motor_number}" />
     </joint>
-    <!-- TODO(ff): not currently set because it's not yet supported -->
-    <!-- <gazebo reference="rotor_${motor_number}_joint"> <axis> <xyz>0 0 1</xyz>
-      <limit> <velocity> ${max_rot_velocity} </velocity> </limit> </axis> </gazebo> -->
-    <link name="rotor_${motor_number}">
+    <link name="blade_link_${motor_number}">
       <inertial>
         <mass value="${mass_rotor}" /> <!-- [kg] -->
@@ -92,5 +60,4 @@
       <visual>
         <geometry>
-          <!-- <cylinder length="0.005" radius="${radius_rotor}"/> --> <!-- [m] -->
           <mesh filename="package://flypulator_description/meshes/${mesh}_${direction}.dae"
             scale="${mesh_scale}" />
@@ -104,35 +71,8 @@
       </collision>
     </link>
+    <!--PX4 memory: attach librotors_gazebo_motor_model to the base_link -->
     <gazebo>
-      <!-- <plugin name="${suffix}_motor_model" filename="librotors_gazebo_motor_model.so"> -->
-      <!--   <robotNamespace>${robot_namespace}</robotNamespace> -->
-      <!--   <jointName>rotor_${motor_number}_joint</jointName> -->
-      <!--   <linkName>rotor_${motor_number}</linkName> -->
-      <!--   <turningDirection>${direction}</turningDirection> -->
-      <!--   <timeConstantUp>${time_constant_up}</timeConstantUp> -->
-      <!--   <timeConstantDown>${time_constant_down}</timeConstantDown> -->
-      <!--   <maxRotVelocity>${max_rot_velocity}</maxRotVelocity> -->
-      <!--   <motorConstant>${motor_constant}</motorConstant> -->
-      <!--   <momentConstant>${moment_constant}</momentConstant> -->
-      <!--   <commandSubTopic>/gazebo/command/motor_speed</commandSubTopic> -->
-      <!--   <motorNumber>${motor_number}</motorNumber> -->
-      <!--   <rotorDragCoefficient>${rotor_drag_coefficient}</rotorDragCoefficient> -->
-      <!--   <rollingMomentCoefficient>${rolling_moment_coefficient}</rollingMomentCoefficient> -->
-      <!--   <motorSpeedPubTopic>/motor_speed/${motor_number}</motorSpeedPubTopic> -->
-      <!--   <rotorVelocitySlowdownSim>${rotor_velocity_slowdown_sim}</rotorVelocitySlowdownSim> -->
-        <!--
-        <gazebo_joint_control_pid>
-          <p>0.1</p>
-          <i>0</i>
-          <d>0</d>
-          <iMax>0</iMax>
-          <iMin>0</iMin>
-          <cmdMax>3</cmdMax>
-          <cmdMin>-3</cmdMin>
-        </gazebo_joint_control_pid>
-      -->
-      <!-- </plugin> -->
-    </gazebo>
-    <gazebo reference="rotor_${motor_number}">
+         </gazebo>
+    <gazebo reference="blade_link_${motor_number}">
       <material>Gazebo/${color}</material>
     </gazebo>
@@ -145,8 +85,5 @@
       <xacro:insert_block name="origin" />
       <axis xyz="0 1 0" />
-      <!-- TODO(ff): not currently set because it's not yet supported -->
-      <!-- <limit effort="2000" velocity="${max_rot_velocity}" /> -->
-      <!-- <limit effort="0" velocity="0" lower="${reflect*0.1745}" upper="${reflect*1.5705}"/> -->
-      <parent link="${parent}" />
+          <parent link="${parent}" />
       <child link="leg_${leg_number}" />
     </joint>
@@ -161,5 +98,4 @@
         <origin xyz="0 0 0" rpy="0 0 0 " />
         <geometry>
-          <!-- <cylinder length="0.005" radius="${radius_rotor}"/> --> <!-- [m] -->
           <mesh filename="package://flypulator_description/meshes/right_leg.dae"
              scale="${mesh_scale}" />
@@ -188,8 +124,5 @@
       <!-- <visual> -->
         <!-- <geometry> -->
-          <!-- <cylinder length="0.005" radius="${radius_rotor}"/> --> <!-- [m] -->
-          <!-- <mesh filename="package://flypulator_description/meshes/${mesh}_${suffix}.dae" -->
-            <!-- scale="${mesh_scale}" /> -->
-            <!-- <cylinder length="${length_leg}" radius="${radius_leg}" />  -->
+<!-- This is not populated as dae shows leg and foot. -->
         <!-- </geometry> -->
       <!-- </visual> -->
@@ -201,33 +134,5 @@
     </link>
     <gazebo>
-      <!-- <plugin name="${suffix}_leg_model" filename="librotors_gazebo_leg_model.so"> -->
-        <!-- <robotNamespace>${robot_namespace}</robotNamespace> -->
-        <!-- <jointName>rotor_${leg_number}_joint</jointName> -->
-        <!-- <linkName>rotor_${leg_number}</linkName> -->
-        <!-- <turningDirection>${direction}</turningDirection> -->
-        <!-- <timeConstantUp>${time_constant_up}</timeConstantUp> -->
-        <!-- <timeConstantDown>${time_constant_down}</timeConstantDown> -->
-        <!-- <maxRotVelocity>${max_rot_velocity}</maxRotVelocity> -->
-        <!-- <legConstant>${leg_constant}</legConstant> -->
-        <!-- <momentConstant>${moment_constant}</momentConstant> -->
-        <!-- <commandSubTopic>/gazebo/command/leg_speed</commandSubTopic> -->
-        <!-- <legNumber>${leg_number}</legNumber> -->
-        <!-- <rotorDragCoefficient>${rotor_drag_coefficient}</rotorDragCoefficient> -->
-        <!-- <rollingMomentCoefficient>${rolling_moment_coefficient}</rollingMomentCoefficient> -->
-        <!-- <motorSpeedPubTopic>/motor_speed/${leg_number}</motorSpeedPubTopic> -->
-        <!-- <rotorVelocitySlowdownSim>${rotor_velocity_slowdown_sim}</rotorVelocitySlowdownSim> -->
-        <!--
-        <gazebo_joint_control_pid>
-          <p>0.1</p>
-          <i>0</i>
-          <d>0</d>
-          <iMax>0</iMax>
-          <iMin>0</iMin>
-          <cmdMax>3</cmdMax>
-          <cmdMin>-3</cmdMin>
-        </gazebo_joint_control_pid>
-      -->
-      <!-- </plugin> -->
-    </gazebo>
+         </gazebo>
     <gazebo reference="leg_${leg_number}">
       <material>Gazebo/${color}</material>

Commit message: cleaning up files

File: flypulator_description/urdf/hexatilt.xacro (robot description, xacro)
@@ -12,5 +12,6 @@
   <!-- Mesh parameters -->
   <xacro:property name="mesh_file" value="hexatilt.dae" />
-  <xacro:property name="mesh_scale" value="0.001 0.001 0.001"/>
+  <!-- <xacro:property name="mesh_scale" value="0.001 0.001 0.001"/> -->
+  <xacro:property name="mesh_scale" value="1 1 1"/>
   <xacro:property name="mesh_scale_prop" value="0.098 0.098 0.098"/>
   <xacro:property name="mesh_scale_leg" value="0.1 0.1 0.1"/>
@@ -262,7 +263,3 @@
     </plugin>
   </gazebo>
-<!-- <gazebo> -->
-<!--     <plugin name="propulsion_plugin_hexa" filename="libpropulsion_plugin_hexa.so"> -->
-<!--     </plugin> -->
-<!--   </gazebo> -->
 </robot>

File: flypulator_description/urdf/multirotor_base.xacro (robot description, xacro)
@@ -73,5 +73,5 @@
     <!--PX4 memory: attach librotors_gazebo_motor_model to the base_link -->
     <gazebo>
-         </gazebo>
+    </gazebo>
     <gazebo reference="blade_link_${motor_number}">
       <material>Gazebo/${color}</material>
