Commit message: cleaning up files

File: flypulator_description/urdf/hexatilt.xacro (robot description, xacro)
@@ -12,5 +12,6 @@
   <!-- Mesh parameters -->
   <xacro:property name="mesh_file" value="hexatilt.dae" />
-  <xacro:property name="mesh_scale" value="0.001 0.001 0.001"/>
+  <!-- <xacro:property name="mesh_scale" value="0.001 0.001 0.001"/> -->
+  <xacro:property name="mesh_scale" value="1 1 1"/>
   <xacro:property name="mesh_scale_prop" value="0.098 0.098 0.098"/>
   <xacro:property name="mesh_scale_leg" value="0.1 0.1 0.1"/>
@@ -45,4 +46,5 @@
   <xacro:property name="leg_pos_side_x" value="0.11" /> <!-- [m] -->
   <xacro:property name="mass_leg" value="0.180" /> <!-- [kg] -->
+  <xacro:include filename="$(find flypulator_description)/urdf/gazebo_plugins.xacro" />
 <!-- Moment of Inertia at Origin   (g mm^2) -->
   <xacro:property name="body_inertia">
@@ -248,21 +250,3 @@
     <xacro:insert_block name="leg_inertia" />
   </xacro:landing_gear>
-<!-- Gazebo plugins .. move to import document.. -->
-  <gazebo>
-    <plugin name="fake_sensor_plugin" filename="libfake_sensor_plugin.so">
-    </plugin>
-  </gazebo>
-  <gazebo>
-    <plugin name="gazebo_ros_control" filename="libgazebo_ros_control.so">
-      <robotNamespace>${namespace}</robotNamespace>
-    </plugin>
-  </gazebo>
-  <gazebo>
-    <plugin name="propulsion_plugin" filename="libpropulsion_plugin.so">
-    </plugin>
-  </gazebo>
-<!-- <gazebo> -->
-<!--     <plugin name="propulsion_plugin_hexa" filename="libpropulsion_plugin_hexa.so"> -->
-<!--     </plugin> -->
-<!--   </gazebo> -->
 </robot>

File: flypulator_description/urdf/hexatilt_base.xacro (robot description, xacro)
@@ -25,6 +25,4 @@
   <!-- macros for gazebo plugins, sensors -->
   <!-- <xacro:include filename="$(find flypulator_description)/urdf/component_snippets.xacro" /> -->
-  <!-- macros for gazebo plugins, for flypulator -->
-  <!-- <xacro:include filename="$(find flypulator_description)/urdf/gazebo_plugins.xacro" /> -->
   <!-- Instantiate hexatilt "mechanics" -->
   <xacro:include filename="$(find flypulator_description)/urdf/hexatilt.xacro" />

Commit message: inital commit to sort out meshes

File: flypulator_description/urdf/hexatilt.xacro (robot description, xacro)
@@ -11,9 +11,9 @@
   <xacro:property name="sqrt2" value="1.4142135623730951" />
   <!-- Mesh parameters -->
-  <xacro:property name="mesh_file" value="hexatilt.dae" />
+  <xacro:property name="mesh_file" value="hexatilt_base_down.dae" />
   <!-- <xacro:property name="mesh_scale" value="0.001 0.001 0.001"/> -->
-  <xacro:property name="mesh_scale" value="1 1 1"/>
-  <xacro:property name="mesh_scale_prop" value="0.098 0.098 0.098"/>
-  <xacro:property name="mesh_scale_leg" value="0.1 0.1 0.1"/>
+  <xacro:property name="mesh_scale" value="0.001 0.001 0.001"/>
+  <xacro:property name="mesh_scale_prop" value="0.001 0.001 0.001"/>
+  <xacro:property name="mesh_scale_leg" value="0.001 0.001 0.001"/>
   <!-- Geometric Parameters -->
   <!-- These parameters are pulled from the .yaml file -->
@@ -45,30 +45,30 @@
   <xacro:property name="base_mass" value="${DP['uav/base_mass']}" /> <!-- [kg] -->
   <xacro:property name="leg_pos_side_x" value="0.11" /> <!-- [m] -->
-  <xacro:property name="mass_leg" value="0.180" /> <!-- [kg] -->
+  <xacro:property name="mass_leg" value="${DP['uav/leg_mass']}"  /> <!-- [kg] -->
   <xacro:include filename="$(find flypulator_description)/urdf/gazebo_plugins.xacro" />
 <!-- Moment of Inertia at Origin   (g mm^2) -->
   <xacro:property name="body_inertia">
     <inertia
-    ixx = "${1.536E+08*to_kgm2}"
-	ixy = "${ 4.372E+04 *to_kgm2}"
-	ixz = "${ 1.475E+04 *to_kgm2}"
-	iyx = "${ 4.372E+04 *to_kgm2}"
-	iyy = "${ 1.580E+08 *to_kgm2}"
-	iyz = "${ -2.790E+04*to_kgm2}"
-	izx = "${ 1.475E+04 *to_kgm2}"
-	izy = "${ -2.790E+04*to_kgm2}"
-	izz = "${ 2.429E+08 *to_kgm2}"     />
+    ixx = "${1.223E+08  *to_kgm2}"
+	ixy = "${-7.268E+04 *to_kgm2}"
+	ixz = "${-1.303E+04 *to_kgm2}"
+	iyx = "${-7.268E+04 *to_kgm2}"
+	iyy = "${1.232E+08  *to_kgm2}"
+	iyz = "${-2.035E+04 *to_kgm2}"
+	izx = "${-1.303E+04 *to_kgm2}"
+	izy = "${-2.035E+04 *to_kgm2}"
+	izz = "${2.355E+08  *to_kgm2}"     />
     </xacro:property>
   <xacro:property name="leg_inertia">
     <inertia
-    ixx = "${ 3.321E+06*to_kgm2 }"
-    ixy = "${ 0.048    *to_kgm2 }"
-    ixz = "${ 4.097E+05*to_kgm2 }"
-    iyx = "${ 0.048    *to_kgm2 }"
-    iyy = "${ 2.407E+06*to_kgm2 }"
-    iyz = "${ -0.271    *to_kgm2 }"
-    izx = "${ 4.097E+05*to_kgm2 }"
-    izy = "${ -0.271   *to_kgm2 }"
-    izz = "${ 1.070E+06*to_kgm2 }"/>
+    ixx = "${ 0*to_kgm2 }"
+    ixy = "${ 0*to_kgm2 }"
+    ixz = "${ 0*to_kgm2 }"
+    iyx = "${ 0*to_kgm2 }"
+    iyy = "${ 0*to_kgm2 }"
+    iyz = "${ 0*to_kgm2 }"
+    izx = "${ 0*to_kgm2 }"
+    izy = "${ 0*to_kgm2 }"
+    izz = "${ 0*to_kgm2 }"/>
      </xacro:property>
   <xacro:property name="rotor_inertia">

File: flypulator_description/urdf/multirotor_base.xacro (robot description, xacro)
@@ -45,4 +45,12 @@
   </xacro:macro>
   <!-- Rotor joint and link -->
+  <!-- The following parameters are artifacts of the gazebo_motor_model plugin. It will be removed when we are sure it is not needed later in SITL integration. -->
+  * motor_constant
+  * moment_constant
+  * time_constant_up
+  * time_constant_down
+  * max_rot_velocity
+  * rotor_drag_coefficient
+  * rolling_moment_coefficient
   <xacro:macro name="vertical_rotor"
     params="robot_namespace suffix direction motor_constant moment_constant parent mass_rotor radius_rotor time_constant_up time_constant_down max_rot_velocity motor_number rotor_drag_coefficient rolling_moment_coefficient color mesh mesh_scale *origin *inertia">
@@ -60,5 +68,5 @@
       <visual>
         <geometry>
-          <mesh filename="package://flypulator_description/meshes/${mesh}_${direction}.dae"
+          <mesh filename="package://flypulator_description/meshes/${direction}.dae"
             scale="${mesh_scale}" />
           <!-- <box size="${2*radius_rotor} 0.01 0.005"/> -->

Commit message: implementing drone with downward facing propellers

File: flypulator_description/urdf/hexatilt.xacro (robot description, xacro)
@@ -12,8 +12,7 @@
   <!-- Mesh parameters -->
   <xacro:property name="mesh_file" value="hexatilt_base_down.dae" />
-  <!-- <xacro:property name="mesh_scale" value="0.001 0.001 0.001"/> -->
-  <xacro:property name="mesh_scale" value="0.001 0.001 0.001"/>
-  <xacro:property name="mesh_scale_prop" value="0.001 0.001 0.001"/>
-  <xacro:property name="mesh_scale_leg" value="0.001 0.001 0.001"/>
+  <xacro:property name="mesh_scale" value="1 1 1"/>
+  <xacro:property name="mesh_scale_prop" value="1 1 1"/>
+  <xacro:property name="mesh_scale_leg" value="1 1 1"/>
   <!-- Geometric Parameters -->
   <!-- These parameters are pulled from the .yaml file -->
@@ -60,4 +59,5 @@
 	izz = "${2.355E+08  *to_kgm2}"     />
     </xacro:property>
+ <!-- The inertia of the legs are set to zero and the MoI of the body includes the legs. -->
   <xacro:property name="leg_inertia">
     <inertia
@@ -100,5 +100,5 @@
   <xacro:vertical_rotor robot_namespace="${namespace}"
     suffix="back_right"
-    direction="cw"
+    direction="ccw"
     motor_constant="${motor_constant}"
     moment_constant="${moment_constant}"
@@ -115,5 +115,5 @@
     mesh_scale="${mesh_scale_prop}"
     color="DarkGrey">
-    <origin xyz="-${arm_length_x+0.01} -${arm_length_y} ${rotor_offset_top}" rpy= "-${rotor_tilt_angle*deg_to_rad} 0  ${60*deg_to_rad}"/>
+    <origin xyz="-${arm_length_x-0.02} -${arm_length_y} ${rotor_offset_top}" rpy= "-${rotor_tilt_angle*deg_to_rad} 0  ${60*deg_to_rad}"/>
     <xacro:insert_block name="rotor_inertia" />
   </xacro:vertical_rotor>
@@ -121,4 +121,24 @@
     robot_namespace="${namespace}"
     suffix="front_right"
+    direction="cw"
+    motor_constant="${motor_constant}"
+    moment_constant="${moment_constant}"
+    parent="base_link"
+    mass_rotor="${mass_rotor}"
+    radius_rotor="${radius_rotor}"
+    time_constant_up="${time_constant_up}"
+    time_constant_down="${time_constant_down}"
+    max_rot_velocity="${max_rot_velocity}"
+    motor_number="2"
+    rotor_drag_coefficient="${rotor_drag_coefficient}"
+    rolling_moment_coefficient="${rolling_moment_coefficient}"
+    mesh="hexatilt_prop"
+    mesh_scale="${mesh_scale_prop}"
+    color="DarkGrey">
+    <origin xyz="${arm_length_x-0.02} -${arm_length_y} ${rotor_offset_top}" rpy="${rotor_tilt_angle*deg_to_rad} 0  ${120*deg_to_rad}" />
+    <xacro:insert_block name="rotor_inertia" />
+  </xacro:vertical_rotor>
+  <xacro:vertical_rotor robot_namespace="${namespace}"
+    suffix="back_right"
     direction="ccw"
     motor_constant="${motor_constant}"
@@ -130,24 +150,4 @@
     time_constant_down="${time_constant_down}"
     max_rot_velocity="${max_rot_velocity}"
-    motor_number="2"
-    rotor_drag_coefficient="${rotor_drag_coefficient}"
-    rolling_moment_coefficient="${rolling_moment_coefficient}"
-    mesh="hexatilt_prop"
-    mesh_scale="${mesh_scale_prop}"
-    color="DarkGrey">
-    <origin xyz="${arm_length_x+0.01} -${arm_length_y} ${rotor_offset_top}" rpy="${rotor_tilt_angle*deg_to_rad} 0  ${120*deg_to_rad}" />
-    <xacro:insert_block name="rotor_inertia" />
-  </xacro:vertical_rotor>
-  <xacro:vertical_rotor robot_namespace="${namespace}"
-    suffix="back_right"
-    direction="cw"
-    motor_constant="${motor_constant}"
-    moment_constant="${moment_constant}"
-    parent="base_link"
-    mass_rotor="${mass_rotor}"
-    radius_rotor="${radius_rotor}"
-    time_constant_up="${time_constant_up}"
-    time_constant_down="${time_constant_down}"
-    max_rot_velocity="${max_rot_velocity}"
     motor_number="3"
     rotor_drag_coefficient="${rotor_drag_coefficient}"
@@ -156,5 +156,5 @@
     mesh_scale="${mesh_scale_prop}"
     color="DarkGrey">
-    <origin xyz="${arm_length_side_x} -${arm_length_side_y} ${rotor_offset_top}" rpy="-${rotor_tilt_angle*deg_to_rad} 0  ${180*deg_to_rad}" />
+    <origin xyz="${arm_length_side_x} +${arm_length_side_y} ${rotor_offset_top}" rpy="-${rotor_tilt_angle*deg_to_rad} 0  ${180*deg_to_rad}" />
     <xacro:insert_block name="rotor_inertia" />
   </xacro:vertical_rotor>
@@ -176,5 +176,5 @@
     mesh_scale="${mesh_scale_prop}"
     color="Red">
-    <origin xyz="${arm_length_x-0.02} ${arm_length_y} ${rotor_offset_top}" rpy= "${rotor_tilt_angle*deg_to_rad} 0  ${240*deg_to_rad}"/>
+    <origin xyz="${arm_length_x-0.0} ${arm_length_y} ${rotor_offset_top}" rpy= "${rotor_tilt_angle*deg_to_rad} 0  ${240*deg_to_rad}"/>
     <xacro:insert_block name="rotor_inertia" />
   </xacro:vertical_rotor>
@@ -197,5 +197,5 @@
     mesh_scale="${mesh_scale_prop}"
     color="Red">
-    <origin xyz="-${arm_length_x-0.02} ${arm_length_y} ${rotor_offset_top}" rpy="-${rotor_tilt_angle*deg_to_rad} 0  -${60*deg_to_rad}" />
+    <origin xyz="-${arm_length_x+0.0} ${arm_length_y} ${rotor_offset_top}" rpy="-${rotor_tilt_angle*deg_to_rad} 0  -${60*deg_to_rad}" />
     <xacro:insert_block name="rotor_inertia" />
   </xacro:vertical_rotor>
@@ -217,5 +217,5 @@
     mesh_scale="${mesh_scale_prop}"
     color="DarkGrey">
-    <origin xyz="-${arm_length_side_x} -${arm_length_side_y} ${rotor_offset_top}" rpy="${rotor_tilt_angle*deg_to_rad} 0  ${0*deg_to_rad}" />
+    <origin xyz="-${arm_length_side_x} +${arm_length_side_y} ${rotor_offset_top}" rpy="${rotor_tilt_angle*deg_to_rad} 0  ${0*deg_to_rad}" />
     <xacro:insert_block name="rotor_inertia" />
   </xacro:vertical_rotor>

File: flypulator_description/urdf/multirotor_base.xacro (robot description, xacro)
@@ -106,5 +106,5 @@
         <origin xyz="0 0 0" rpy="0 0 0 " />
         <geometry>
-          <mesh filename="package://flypulator_description/meshes/right_leg.dae"
+          <mesh filename="package://flypulator_description/meshes/leg.dae"
              scale="${mesh_scale}" />
             <!-- <cylinder length="${length_leg}" radius="${radius_leg}" /> <1 [m] -1> -->

Commit message: corrected TFs and motor numbering

File: flypulator_description/urdf/hexatilt.xacro (robot description, xacro)
@@ -43,5 +43,5 @@
  <!-- Mass and inertial Properties -->
   <xacro:property name="base_mass" value="${DP['uav/base_mass']}" /> <!-- [kg] -->
-  <xacro:property name="leg_pos_side_x" value="0.11" /> <!-- [m] -->
+  <xacro:property name="leg_pos_side_y" value="0.11" /> <!-- [m] -->
   <xacro:property name="mass_leg" value="${DP['uav/leg_mass']}"  /> <!-- [kg] -->
   <xacro:include filename="$(find flypulator_description)/urdf/gazebo_plugins.xacro" />
@@ -98,27 +98,27 @@
   </xacro:multirotor_base_macro>
   <!-- Instantiate rotors -->
-  <xacro:vertical_rotor robot_namespace="${namespace}"
-    suffix="back_right"
-    direction="ccw"
-    motor_constant="${motor_constant}"
-    moment_constant="${moment_constant}"
-    parent="base_link"
-    mass_rotor="${mass_rotor}"
-    radius_rotor="${radius_rotor}"
-    time_constant_up="${time_constant_up}"
-    time_constant_down="${time_constant_down}"
-    max_rot_velocity="${max_rot_velocity}"
-    motor_number="1"
-    rotor_drag_coefficient="${rotor_drag_coefficient}"
-    rolling_moment_coefficient="${rolling_moment_coefficient}"
-    mesh="hexatilt_prop"
-    mesh_scale="${mesh_scale_prop}"
-    color="DarkGrey">
-    <origin xyz="-${arm_length_x-0.02} -${arm_length_y} ${rotor_offset_top}" rpy= "-${rotor_tilt_angle*deg_to_rad} 0  ${60*deg_to_rad}"/>
-    <xacro:insert_block name="rotor_inertia" />
-  </xacro:vertical_rotor>
  <xacro:vertical_rotor
     robot_namespace="${namespace}"
     suffix="front_right"
+    direction="ccw"
+    motor_constant="${motor_constant}"
+    moment_constant="${moment_constant}"
+    parent="base_link"
+    mass_rotor="${mass_rotor}"
+    radius_rotor="${radius_rotor}"
+    time_constant_up="${time_constant_up}"
+    time_constant_down="${time_constant_down}"
+    max_rot_velocity="${max_rot_velocity}"
+    motor_number="1"
+    rotor_drag_coefficient="${rotor_drag_coefficient}"
+    rolling_moment_coefficient="${rolling_moment_coefficient}"
+    mesh="hexatilt_prop"
+    mesh_scale="${mesh_scale_prop}"
+    color="Red">
+    <origin xyz="${arm_length_x-0.0} -${arm_length_y-0.02} ${rotor_offset_top}" rpy="-${rotor_tilt_angle*deg_to_rad} 0  ${150*deg_to_rad}" />
+    <xacro:insert_block name="rotor_inertia" />
+  </xacro:vertical_rotor>
+  <xacro:vertical_rotor robot_namespace="${namespace}"
+    suffix="front_left"
     direction="cw"
     motor_constant="${motor_constant}"
@@ -135,6 +135,6 @@
     mesh="hexatilt_prop"
     mesh_scale="${mesh_scale_prop}"
-    color="DarkGrey">
-    <origin xyz="${arm_length_x-0.02} -${arm_length_y} ${rotor_offset_top}" rpy="${rotor_tilt_angle*deg_to_rad} 0  ${120*deg_to_rad}" />
+    color="Red">
+    <origin xyz="${arm_length_x-0.0} ${arm_length_y-0.02} ${rotor_offset_top}" rpy= "${rotor_tilt_angle*deg_to_rad} 0  ${210*deg_to_rad}"/>
     <xacro:insert_block name="rotor_inertia" />
   </xacro:vertical_rotor>
@@ -156,25 +156,5 @@
     mesh_scale="${mesh_scale_prop}"
     color="DarkGrey">
-    <origin xyz="${arm_length_side_x} +${arm_length_side_y} ${rotor_offset_top}" rpy="-${rotor_tilt_angle*deg_to_rad} 0  ${180*deg_to_rad}" />
-    <xacro:insert_block name="rotor_inertia" />
-  </xacro:vertical_rotor>
-  <xacro:vertical_rotor robot_namespace="${namespace}"
-    suffix="front_left"
-    direction="cw"
-    motor_constant="${motor_constant}"
-    moment_constant="${moment_constant}"
-    parent="base_link"
-    mass_rotor="${mass_rotor}"
-    radius_rotor="${radius_rotor}"
-    time_constant_up="${time_constant_up}"
-    time_constant_down="${time_constant_down}"
-    max_rot_velocity="${max_rot_velocity}"
-    motor_number="4"
-    rotor_drag_coefficient="${rotor_drag_coefficient}"
-    rolling_moment_coefficient="${rolling_moment_coefficient}"
-    mesh="hexatilt_prop"
-    mesh_scale="${mesh_scale_prop}"
-    color="Red">
-    <origin xyz="${arm_length_x-0.0} ${arm_length_y} ${rotor_offset_top}" rpy= "${rotor_tilt_angle*deg_to_rad} 0  ${240*deg_to_rad}"/>
+    <origin xyz="-${arm_length_side_x} +${arm_length_side_y} ${rotor_offset_top}" rpy="-${rotor_tilt_angle*deg_to_rad} 0  -${90*deg_to_rad}" />
     <xacro:insert_block name="rotor_inertia" />
   </xacro:vertical_rotor>
@@ -182,4 +162,24 @@
     robot_namespace="${namespace}"
     suffix="back_left"
+    direction="cw"
+    motor_constant="${motor_constant}"
+    moment_constant="${moment_constant}"
+    parent="base_link"
+    mass_rotor="${mass_rotor}"
+    radius_rotor="${radius_rotor}"
+    time_constant_up="${time_constant_up}"
+    time_constant_down="${time_constant_down}"
+    max_rot_velocity="${max_rot_velocity}"
+    motor_number="4"
+    rotor_drag_coefficient="${rotor_drag_coefficient}"
+    rolling_moment_coefficient="${rolling_moment_coefficient}"
+    mesh="hexatilt_prop"
+    mesh_scale="${mesh_scale_prop}"
+    color="DarkGrey">
+    <origin xyz="-${arm_length_x+0.0} ${arm_length_y} ${rotor_offset_top}" rpy="${rotor_tilt_angle*deg_to_rad} 0  -${30*deg_to_rad}" />
+    <xacro:insert_block name="rotor_inertia" />
+  </xacro:vertical_rotor>
+  <xacro:vertical_rotor robot_namespace="${namespace}"
+    suffix="back_right"
     direction="ccw"
     motor_constant="${motor_constant}"
@@ -196,6 +196,6 @@
     mesh="hexatilt_prop"
     mesh_scale="${mesh_scale_prop}"
-    color="Red">
-    <origin xyz="-${arm_length_x+0.0} ${arm_length_y} ${rotor_offset_top}" rpy="-${rotor_tilt_angle*deg_to_rad} 0  -${60*deg_to_rad}" />
+    color="DarkGrey">
+    <origin xyz="-${arm_length_x-0.0} -${arm_length_y} ${rotor_offset_top}" rpy= "-${rotor_tilt_angle*deg_to_rad} 0  ${30*deg_to_rad}"/>
     <xacro:insert_block name="rotor_inertia" />
   </xacro:vertical_rotor>
@@ -217,5 +217,5 @@
     mesh_scale="${mesh_scale_prop}"
     color="DarkGrey">
-    <origin xyz="-${arm_length_side_x} +${arm_length_side_y} ${rotor_offset_top}" rpy="${rotor_tilt_angle*deg_to_rad} 0  ${0*deg_to_rad}" />
+    <origin xyz="-${arm_length_side_x} -${arm_length_side_y} ${rotor_offset_top}" rpy="${rotor_tilt_angle*deg_to_rad} 0  ${90*deg_to_rad}" />
     <xacro:insert_block name="rotor_inertia" />
   </xacro:vertical_rotor>
@@ -232,5 +232,5 @@
     color="DarkGrey"
     reflect="-1">
-    <origin xyz="${leg_pos_side_x} 0 -0.02" rpy="0 -${10*deg_to_rad} 0" />
+    <origin xyz="0 ${leg_pos_side_y} -0.02" rpy="0 ${10*deg_to_rad} -${90*deg_to_rad}" />
     <xacro:insert_block name="leg_inertia" />
   </xacro:landing_gear>
@@ -247,5 +247,5 @@
     reflect="1"
     color="DarkGrey">
-    <origin xyz="-${leg_pos_side_x} 0 -0.02" rpy="0 ${10*deg_to_rad} 0" />
+    <origin xyz="0 -${leg_pos_side_y} -0.02" rpy="0 ${10*deg_to_rad} ${90*deg_to_rad}" />
     <xacro:insert_block name="leg_inertia" />
   </xacro:landing_gear>

File: flypulator_description/urdf/multirotor_base.xacro (robot description, xacro)
@@ -13,5 +13,5 @@
     <link name="base_link"></link>
     <joint name="base_joint" type="fixed">
-      <origin xyz="0 0 0" rpy="0 0 0" />
+        <origin xyz="0 0 0" rpy="0 0 ${0*deg_to_rad}" />
       <parent link="base_link" />
       <child link="base_link_inertia" />
@@ -24,5 +24,5 @@
       </inertial>
       <visual>
-        <origin xyz="0 0 0" rpy="0 0 0" />
+        <origin xyz="0 0 0" rpy="0 0 ${90*deg_to_rad}" />
         <geometry>
           <mesh filename="package://flypulator_description/meshes/${mesh_file}"
