Commit message: some adaption in urdf model.

File: flypulator_description/urdf/hexatilt.xacro (robot description, xacro)
@@ -17,32 +17,23 @@
   <!-- Geometric Parameters -->
   <!-- These parameters are pulled from the .yaml file -->
-  <xacro:property name="rotor_tilt_angle"   value="${DP['uav/alpha']}"/> <!--in [deg]-->
-  <xacro:property name="body_radius"        value="${DP['uav/base_radius']}" /> <!-- [m] -->
-  <xacro:property name="body_height"        value="${DP['uav/base_height']}" />
-  <xacro:property name="mass_rotor"         value="${DP['uav/blade_mass']}" /> <!-- [kg] -->
-  <xacro:property name="arm_length_x"       value="${DP['uav/x']}" /> <!-- [Man[m] -->
-  <xacro:property name="arm_length_y"       value="${DP['uav/y']}" /> <!-- [m] -->
-  <xacro:property name="arm_length_side_x"  value="${DP['uav/side_x']}" /> <!-- [m] -->
-  <xacro:property name="arm_length_side_y"  value="${DP['uav/side_y']}" /> <!-- [m] -->
-  <xacro:property name="radius_leg"         value="${DP['uav/leg_radius']}" /> <!--[Man [m] -->
-  <xacro:property name="length_leg"         value="${DP['uav/leg_length']}" /> <!-- [m] -->
-  <xacro:property name="rotor_offset_top"   value="${DP['uav/blade_offset_top']}"/> <!-- [m] -->
-  <xacro:property name="radius_rotor"       value="${DP['uav/blade_radius']}" /> <!-- [[Manm] -->
+  <xacro:property name="base_mass" 			value="${DP['urdf/base_mass']}" /> <!-- [kg] -->
+  <xacro:property name="rotor_tilt_angle"   value="${DP['urdf/alpha']}"/> <!--in [deg]-->
+  <xacro:property name="body_radius"        value="${DP['urdf/base_radius']}" /> <!-- [m] -->
+  <xacro:property name="body_height"        value="${DP['urdf/base_height']}" />
+  <xacro:property name="mass_prop"         	value="${DP['urdf/propeller_mass']}" /> <!-- [kg] -->
+  <xacro:property name="arm_length"       	value="${DP['urdf/arm_length']}" /> <!-- [m] -->
+  <xacro:property name="radius_leg"         value="${DP['urdf/leg_radius']}" /> <!--[m] -->
+  <xacro:property name="length_leg"         value="${DP['urdf/leg_length']}" /> <!-- [m] -->
+  <xacro:property name="mass_leg" 			value="${DP['urdf/leg_mass']}"  /> <!-- [kg] -->
+  <xacro:property name="rotor_offset_top"   value="${DP['urdf/propeller_offset_top']}"/> <!-- [m] -->
+  <xacro:property name="radius_rotor"       value="${DP['urdf/propeller_radius']}" /> <!-- [m] -->
    <!-- Simulation Properties -->
   <xacro:property name="max_leg_velocity" value="0.10" /> <!-- [m] -->
   <xacro:property name="rotor_velocity_slowdown_sim" value="10" />
-  <xacro:property name="motor_constant" value="8.54858e-06" /> <!-- [kg.m/s^2] -->
-  <xacro:property name="moment_constant" value="0.06" /> <!-- [m] -->
-  <xacro:property name="time_constant_up" value="0.0125" /> <!-- [s] -->
-  <xacro:property name="time_constant_down" value="0.025" /> <!-- [s] -->
   <xacro:property name="max_rot_velocity" value="1100" /> <!-- [rad/s] -->
-  <xacro:property name="rotor_drag_coefficient" value="8.06428e-04" />
-  <xacro:property name="rolling_moment_coefficient" value="0.000001" />
   <xacro:property name="color" value="DarkGrey" />
   <!-- Property Blocks -->
  <!-- Mass and inertial Properties -->
-  <xacro:property name="base_mass" value="${DP['uav/base_mass']}" /> <!-- [kg] -->
   <xacro:property name="leg_pos_side_y" value="0.11" /> <!-- [m] -->
-  <xacro:property name="mass_leg" value="${DP['uav/leg_mass']}"  /> <!-- [kg] -->
   <xacro:include filename="$(find flypulator_description)/urdf/gazebo_plugins.xacro" />
 <!-- Moment of Inertia at Origin   (g mm^2) -->
@@ -98,23 +89,18 @@
   </xacro:multirotor_base_macro>
   <!-- Instantiate rotors -->
+  <!-- suffix, max_rot_velocity, mesh are currently unused. -->
  <xacro:vertical_rotor
     robot_namespace="${namespace}"
     suffix="front_right"
     direction="ccw"
-    motor_constant="${motor_constant}"
-    moment_constant="${moment_constant}"
-    parent="base_link"
-    mass_rotor="${mass_rotor}"
-    radius_rotor="${radius_rotor}"
-    time_constant_up="${time_constant_up}"
-    time_constant_down="${time_constant_down}"
+    parent="base_link"
+    mass_propeller="${mass_prop}"
+    radius_rotor="${radius_rotor}"
     max_rot_velocity="${max_rot_velocity}"
     motor_number="1"
-    rotor_drag_coefficient="${rotor_drag_coefficient}"
-    rolling_moment_coefficient="${rolling_moment_coefficient}"
     mesh="hexatilt_prop"
     mesh_scale="${mesh_scale_prop}"
     color="Red">
-    <origin xyz="${arm_length_x-0.0} -${arm_length_y-0.02} ${rotor_offset_top}" rpy="-${rotor_tilt_angle*deg_to_rad} 0  ${150*deg_to_rad}" />
+    <origin xyz="${arm_length*cos30} -${arm_length*sin30} ${rotor_offset_top}" rpy="-${rotor_tilt_angle*deg_to_rad} 0  ${150*deg_to_rad}" />
     <xacro:insert_block name="rotor_inertia" />
   </xacro:vertical_rotor>
@@ -122,39 +108,27 @@
     suffix="front_left"
     direction="cw"
-    motor_constant="${motor_constant}"
-    moment_constant="${moment_constant}"
-    parent="base_link"
-    mass_rotor="${mass_rotor}"
-    radius_rotor="${radius_rotor}"
-    time_constant_up="${time_constant_up}"
-    time_constant_down="${time_constant_down}"
+    parent="base_link"
+    mass_propeller="${mass_prop}"
+    radius_rotor="${radius_rotor}"
     max_rot_velocity="${max_rot_velocity}"
     motor_number="2"
-    rotor_drag_coefficient="${rotor_drag_coefficient}"
-    rolling_moment_coefficient="${rolling_moment_coefficient}"
     mesh="hexatilt_prop"
     mesh_scale="${mesh_scale_prop}"
     color="Red">
-    <origin xyz="${arm_length_x-0.0} ${arm_length_y-0.02} ${rotor_offset_top}" rpy= "${rotor_tilt_angle*deg_to_rad} 0  ${210*deg_to_rad}"/>
-    <xacro:insert_block name="rotor_inertia" />
-  </xacro:vertical_rotor>
-  <xacro:vertical_rotor robot_namespace="${namespace}"
-    suffix="back_right"
+    <origin xyz="${arm_length*cos30} ${arm_length*sin30} ${rotor_offset_top}" rpy= "${rotor_tilt_angle*deg_to_rad} 0  ${210*deg_to_rad}"/>
+    <xacro:insert_block name="rotor_inertia" />
+  </xacro:vertical_rotor>
+  <xacro:vertical_rotor robot_namespace="${namespace}"
+    suffix="left"
     direction="ccw"
-    motor_constant="${motor_constant}"
-    moment_constant="${moment_constant}"
-    parent="base_link"
-    mass_rotor="${mass_rotor}"
-    radius_rotor="${radius_rotor}"
-    time_constant_up="${time_constant_up}"
-    time_constant_down="${time_constant_down}"
+    parent="base_link"
+    mass_propeller="${mass_prop}"
+    radius_rotor="${radius_rotor}"
     max_rot_velocity="${max_rot_velocity}"
     motor_number="3"
-    rotor_drag_coefficient="${rotor_drag_coefficient}"
-    rolling_moment_coefficient="${rolling_moment_coefficient}"
-    mesh="hexatilt_prop"
-    mesh_scale="${mesh_scale_prop}"
-    color="DarkGrey">
-    <origin xyz="-${arm_length_side_x} +${arm_length_side_y} ${rotor_offset_top}" rpy="-${rotor_tilt_angle*deg_to_rad} 0  -${90*deg_to_rad}" />
+    mesh="hexatilt_prop"
+    mesh_scale="${mesh_scale_prop}"
+    color="DarkGrey">
+    <origin xyz="0 ${arm_length} ${rotor_offset_top}" rpy="-${rotor_tilt_angle*deg_to_rad} 0  -${90*deg_to_rad}" />
     <xacro:insert_block name="rotor_inertia" />
   </xacro:vertical_rotor>
@@ -163,19 +137,13 @@
     suffix="back_left"
     direction="cw"
-    motor_constant="${motor_constant}"
-    moment_constant="${moment_constant}"
-    parent="base_link"
-    mass_rotor="${mass_rotor}"
-    radius_rotor="${radius_rotor}"
-    time_constant_up="${time_constant_up}"
-    time_constant_down="${time_constant_down}"
+    parent="base_link"
+    mass_propeller="${mass_prop}"
+    radius_rotor="${radius_rotor}"
     max_rot_velocity="${max_rot_velocity}"
     motor_number="4"
-    rotor_drag_coefficient="${rotor_drag_coefficient}"
-    rolling_moment_coefficient="${rolling_moment_coefficient}"
-    mesh="hexatilt_prop"
-    mesh_scale="${mesh_scale_prop}"
-    color="DarkGrey">
-    <origin xyz="-${arm_length_x+0.0} ${arm_length_y} ${rotor_offset_top}" rpy="${rotor_tilt_angle*deg_to_rad} 0  -${30*deg_to_rad}" />
+    mesh="hexatilt_prop"
+    mesh_scale="${mesh_scale_prop}"
+    color="DarkGrey">
+    <origin xyz="-${arm_length*cos30} ${arm_length*sin30} ${rotor_offset_top}" rpy="${rotor_tilt_angle*deg_to_rad} 0  -${30*deg_to_rad}" />
     <xacro:insert_block name="rotor_inertia" />
   </xacro:vertical_rotor>
@@ -183,39 +151,27 @@
     suffix="back_right"
     direction="ccw"
-    motor_constant="${motor_constant}"
-    moment_constant="${moment_constant}"
-    parent="base_link"
-    mass_rotor="${mass_rotor}"
-    radius_rotor="${radius_rotor}"
-    time_constant_up="${time_constant_up}"
-    time_constant_down="${time_constant_down}"
+    parent="base_link"
+    mass_propeller="${mass_prop}"
+    radius_rotor="${radius_rotor}"
     max_rot_velocity="${max_rot_velocity}"
     motor_number="5"
-    rotor_drag_coefficient="${rotor_drag_coefficient}"
-    rolling_moment_coefficient="${rolling_moment_coefficient}"
-    mesh="hexatilt_prop"
-    mesh_scale="${mesh_scale_prop}"
-    color="DarkGrey">
-    <origin xyz="-${arm_length_x-0.0} -${arm_length_y} ${rotor_offset_top}" rpy= "-${rotor_tilt_angle*deg_to_rad} 0  ${30*deg_to_rad}"/>
-    <xacro:insert_block name="rotor_inertia" />
-  </xacro:vertical_rotor>
-  <xacro:vertical_rotor robot_namespace="${namespace}"
-    suffix="back_right"
+    mesh="hexatilt_prop"
+    mesh_scale="${mesh_scale_prop}"
+    color="DarkGrey">
+    <origin xyz="-${arm_length*cos30} -${arm_length*sin30} ${rotor_offset_top}" rpy= "-${rotor_tilt_angle*deg_to_rad} 0  ${30*deg_to_rad}"/>
+    <xacro:insert_block name="rotor_inertia" />
+  </xacro:vertical_rotor>
+  <xacro:vertical_rotor robot_namespace="${namespace}"
+    suffix="right"
     direction="cw"
-    motor_constant="${motor_constant}"
-    moment_constant="${moment_constant}"
-    parent="base_link"
-    mass_rotor="${mass_rotor}"
-    radius_rotor="${radius_rotor}"
-    time_constant_up="${time_constant_up}"
-    time_constant_down="${time_constant_down}"
+    parent="base_link"
+    mass_propeller="${mass_prop}"
+    radius_rotor="${radius_rotor}"
     max_rot_velocity="${max_rot_velocity}"
     motor_number="6"
-    rotor_drag_coefficient="${rotor_drag_coefficient}"
-    rolling_moment_coefficient="${rolling_moment_coefficient}"
-    mesh="hexatilt_prop"
-    mesh_scale="${mesh_scale_prop}"
-    color="DarkGrey">
-    <origin xyz="-${arm_length_side_x} -${arm_length_side_y} ${rotor_offset_top}" rpy="${rotor_tilt_angle*deg_to_rad} 0  ${90*deg_to_rad}" />
+    mesh="hexatilt_prop"
+    mesh_scale="${mesh_scale_prop}"
+    color="DarkGrey">
+    <origin xyz="0 -${arm_length} ${rotor_offset_top}" rpy="${rotor_tilt_angle*deg_to_rad} 0  ${90*deg_to_rad}" />
     <xacro:insert_block name="rotor_inertia" />
   </xacro:vertical_rotor>

File: flypulator_description/urdf/multirotor_base.xacro (robot description, xacro)
@@ -37,7 +37,4 @@
       </collision>
     </link>
-    <!--PX4 memory: attach multirotor_base_plugin to the base_link -->
-    <gazebo>
-    </gazebo>
     <gazebo reference="base_link">
     <material>Gazebo/${color}</material>
@@ -54,5 +51,5 @@
   * rolling_moment_coefficient
   <xacro:macro name="vertical_rotor"
-    params="robot_namespace suffix direction motor_constant moment_constant parent mass_rotor radius_rotor time_constant_up time_constant_down max_rot_velocity motor_number rotor_drag_coefficient rolling_moment_coefficient color mesh mesh_scale *origin *inertia">
+    params="robot_namespace suffix direction parent mass_propeller radius_rotor max_rot_velocity motor_number color mesh mesh_scale *origin *inertia">
     <joint name="blade_joint_${motor_number}" type="continuous">
       <xacro:insert_block name="origin" />
@@ -63,5 +60,5 @@
     <link name="blade_link_${motor_number}">
       <inertial>
-        <mass value="${mass_rotor}" /> <!-- [kg] -->
+        <mass value="${mass_propeller}" /> <!-- [kg] -->
         <xacro:insert_block name="inertia" />
       </inertial>
@@ -79,7 +76,4 @@
       </collision>
     </link>
-    <!--PX4 memory: attach librotors_gazebo_motor_model to the base_link -->
-    <gazebo>
-    </gazebo>
     <gazebo reference="blade_link_${motor_number}">
       <material>Gazebo/${color}</material>
@@ -90,12 +84,12 @@
     params="robot_namespace suffix reflect parent mass_leg radius_leg length_leg max_leg_velocity leg_number color mesh mesh_scale *origin *inertia">
 <!-- Landing gear joint: -->
-    <joint name="leg_${leg_number}_joint" type="fixed">
+    <joint name="leg_joint_${leg_number}" type="fixed">
       <xacro:insert_block name="origin" />
       <axis xyz="0 1 0" />
           <parent link="${parent}" />
-      <child link="leg_${leg_number}" />
+      <child link="leg_link_${leg_number}" />
     </joint>
 <!-- Leg link -->
-    <link name="leg_${leg_number}">
+    <link name="leg_link_${leg_number}">
       <inertial>
         <origin xyz="0 0 -${length_leg/2}" rpy="0 0 0 " />
@@ -119,11 +113,11 @@
     </link>
 <!-- Joint Leg-foot fixed -->
-    <joint name="foot_${leg_number}_joint" type="fixed">
-      <parent link="leg_${leg_number}" />
-      <child link="foot_${leg_number}" />
+    <joint name="foot_joint_${leg_number}" type="fixed">
+      <parent link="leg_link_${leg_number}" />
+      <child link="foot_link_${leg_number}" />
       <origin xyz="0 0 -${length_leg}" rpy= "1.57 0 0"/>
     </joint>
 <!-- Foot link -->
-    <link name="foot_${leg_number}">
+    <link name="foot_link_${leg_number}">
       <inertial>
         <mass value="${mass_leg}" /> <!-- [kg] -->
@@ -141,7 +135,5 @@
       </collision>
     </link>
-    <gazebo>
-         </gazebo>
-    <gazebo reference="leg_${leg_number}">
+    <gazebo reference="leg_link_${leg_number}">
       <material>Gazebo/${color}</material>
     </gazebo>
